Commit message: new cad, deleted rear ball, replaced with left and right leg

File: robots/legacy/old1_full_assembly_robot_unit.urdf (robot description, URDF)
Before this commit: robot full_assembly_robot_unit, 7 links, 6 joints
Links:
- removed link left_leg_link
- removed link right_leg_link
- added link rear_ball_link, mass 0.005; collision mesh filename=robots/meshes/rear_ball_link.STL; visual mesh filename=robots/meshes/rear_ball_link.STL
Joints:
- removed joint left_leg_joint
- removed joint right_leg_joint
- added joint rear_ball_joint: type continuous, parent chassis_link, child rear_ball_link, origin xyz=0 0.0061 0.00503 rpy=3.1416 -1.5708 0, axis 1 0 0
