Commit message: changed height btw chassis and ground

File: robots/legacy/old2_full_assembly_robot_unit.urdf (robot description, URDF)
Before this commit: robot full_assembly_robot_unit, 7 links, 6 joints
Links:
- link left_wheel_link: geometry collision cylinder length=0.001 radius=0.00575; visual mesh filename=robots/meshes/left_wheel_link.STL
- link right_wheel_link: geometry collision cylinder length=0.001 radius=0.00575; visual mesh filename=robots/meshes/right_wheel_link.STL
Joints:
- joint left_leg_joint: origin xyz=0.014 0.0143 0.0173 rpy=-1.5708 0 3.1416 -> xyz=0.014 0.0113 0.0173 rpy=-1.5708 0 3.1416
- joint left_wheel_joint: origin xyz=0.02264 0.009 -0.02193 rpy=0 0 0 -> xyz=0.02264 0.0061 -0.02193 rpy=0 0 0
- joint right_leg_joint: origin xyz=-0.014 0.0143 0.0173 rpy=-1.5708 0 3.1416 -> xyz=-0.014 0.0113 0.0173 rpy=-1.5708 0 3.1416
- joint right_wheel_joint: origin xyz=-0.02264 0.009 -0.02193 rpy=3.1416 0 3.1416 -> xyz=-0.02264 0.0061 -0.02193 rpy=3.1416 0 3.1416
